File: Electronics/LogicAnalyzer/LevelShifter/LevelShifter.kicad_pcb (KiCad board)
At the start: 2 copper layers, 28.3 x 39.8 mm, 20 parts, among them J1 Conn_02x15_Odd_Even, J2 Conn_02x15_Odd_Even, U1 TXU0104PWR, U2 TXU0104PWR, U3 TXU0104PWR, U4 TXU0104PWR, U5 TXU0104PWR, U6 TXU0104PWR

Commit message: WIP Changes
Other:
- board text added: "< To probes"
- board text added: "From Logic Analyzer >"
- board text removed: "This side UP"
